File: simpleLED/simpleLED.kicad_pcb (KiCad board)
At the start: 2 copper layers, 9 parts, among them SW1 SW_MEC_5G, SW2 SW_MEC_5G, SW3 SW_MEC_5G

Commit message: updated
Parts:
- removed D2, D3: LED, Diode_SMD:D_1210_3225Metric_Pad1.42x2.65mm_HandSolder
- removed R2, R3: R, Resistor_THT:R_Axial_DIN0204_L3.6mm_D1.6mm_P1.90mm_Vertical
- removed SW2, SW3: SW_MEC_5G, Button_Switch_SMD:SW_SPST_Omron_B3FS-100xP
- added J1: USB_A, simpleLED:USB-A-Male, F.Cu at (78.5, 35.0)
- R1: footprint Resistor_THT:R_Axial_DIN0204_L3.6mm_D1.6mm_P1.90mm_Vertical -> Resistor_THT:R_Axial_DIN0204_L3.6mm_D1.6mm_P5.08mm_Horizontal
- SW1: value SW_MEC_5G -> SW_Push; footprint Button_Switch_SMD:SW_SPST_Omron_B3FS-100xP -> Button_Switch_SMD:SW_SPST_PTS645
- moved SW1 81.9 mm to (64.0, 39.0)
- moved D1 74.1 mm to (67.0, 47.0), turned to 90 degrees
- moved R1 72.0 mm to (61.0, 45.0), turned to -90 degrees
Connections:
- SW1 pad 2: +5V -> Net-(R1-Pad1)
Other:
- board outline added: 28 x 18 mm

Commit message: updated
Parts:
- removed D1: LED, Diode_SMD:D_1210_3225Metric_Pad1.42x2.65mm_HandSolder
- added LED1: LED, Diode_SMD:D_1210_3225Metric_Pad1.42x2.65mm_HandSolder, F.Cu at (50.2, 32.5)
- added REF**: ruler, simpleLED:ruler, F.Cu at (71.5, 25.8)
- added REF**: MountingHole_3.2mm_M3, MountingHole:MountingHole_3.2mm_M3, F.Cu at (115.2, 36.0)
- moved J1 54.3 mm to (24.2, 33.5), turned to 0 degrees
- moved SW1 24.7 mm to (39.8, 34.5), turned to 180 degrees
- moved R1 15.5 mm to (47.7, 37.0), turned to 0 degrees
Routing:
- net GND: track 0.00 -> 26.2 mm, vias 0 -> 2
- net +5V: track 0.00 -> 19.1 mm
- net Net-(R1-Pad1): track 0.00 -> 16.0 mm
- net Net-(D1-Pad2): track 0.00 -> 4.94 mm
Other:
- board size 28 x 18 mm -> 100 x 20 mm
- board text added: "National Institute of Technology, Kagawa College"

Commit message: updated
Routing:
- added copper zone on F.Cu, net +5V
- added copper zone on B.Cu, net GND
Changed lines of the file:
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@@
       (effects (font (size 1 1) (thickness 0.15)))
     )
-    (fp_rect (start -5.5 -6) (end 5.5 6) (layer "F.SilkS") (width 0.12) (fill none))
+    (fp_rect (start -5.5 -6) (end 5.5 6) (layer "F.Fab") (width 0.12) (fill none))
     (pad "1" smd roundrect (at 0.5 3.5) (size 10 1.5) (layers "F.Cu" "F.Paste" "F.Mask") (roundrect_rratio 0.25)
       (net 1 "+5V") (pinfunction "VBUS") (pintype "power_in"))
@@
   (segment (start 51.7375 32.5) (end 51.7375 34.4875) (width 0.5) (layer "F.Cu") (net 6))
   (segment (start 52.79 35.54) (end 52.79 37) (width 0.5) (layer "F.Cu") (net 6))
+  (zone (net 1) (net_name "+5V") (layer "F.Cu") (hatch edge 0.508)
+    (connect_pads (clearance 0.508))
+    (min_thickness 0.254) (filled_areas_thickness no)
+    (fill yes (thermal_gap 0.508) (thermal_bridge_width 0.508))
+    (polygon
+      (pts
+        (xy 55 39.5)
+        (xy 30 39.5)
+        (xy 30 27.5)
+        (xy 55 27.5)
+      )
+    )
+  )
+  (zone (net 4) (net_name "GND") (layer "B.Cu") (hatch edge 0.508)
+    (connect_pads (clearance 0.508))
+    (min_thickness 0.254) (filled_areas_thickness no)
+    (fill yes (thermal_gap 0.508) (thermal_bridge_width 0.508))
+    (polygon
+      (pts
+        (xy 55 39.5)
+        (xy 30 39.5)
+        (xy 30 27.5)
+        (xy 55 27.5)
+      )
+    )
+  )
 )

Commit message: updated
Parts:
- removed J1: USB_A, simpleLED:USB-A-Male
- removed LED1: LED, Diode_SMD:D_1210_3225Metric_Pad1.42x2.65mm_HandSolder
- removed R1: R, Resistor_THT:R_Axial_DIN0204_L3.6mm_D1.6mm_P5.08mm_Horizontal
- removed SW1: SW_Push, Button_Switch_SMD:SW_SPST_PTS645
- added LED: LED, LED_THT:LED_D3.0mm, F.Cu at (45.7, 31.5)
- added R: R, Resistor_THT:R_Axial_DIN0204_L3.6mm_D1.6mm_P7.62mm_Horizontal, F.Cu at (43.4, 37.0)
- added SW: SW_Push, Button_Switch_THT:SW_PUSH_6mm, F.Cu at (34.0, 37.0)
- added USB: USB_A, simpleLED:USB-A-Male, F.Cu at (24.2, 33.5)
Routing:
- net Net-(R1-Pad1): track 16.0 -> 11.4 mm
- net GND: track 26.2 -> 22.3 mm, vias 2 -> 1
- net +5V: track 19.1 -> 15.8 mm
- net Net-(D1-Pad2): track 4.94 -> 7.82 mm
Other:
- board text added: "+"
- board text added: "National Institute of Technology, Kagawa College Department of Electronic Systems Engineering"
- board text removed: "National Institute of Technology, Kagawa College"
