File: simpleLED/simpleLED.kicad_sch (KiCad schematic)
At the start: 9 parts, among them SW1 SW_MEC_5G, SW2 SW_MEC_5G, SW3 SW_MEC_5G

Commit message: updated
Parts:
- removed D2, D3: LED, Diode_SMD:D_1210_3225Metric_Pad1.42x2.65mm_HandSolder, symbol Device:LED
- removed R2, R3: R, Resistor_THT:R_Axial_DIN0204_L3.6mm_D1.6mm_P1.90mm_Vertical, symbol Device:R
- removed SW1, SW2, SW3: SW_MEC_5G, Button_Switch_SMD:SW_SPST_Omron_B3FS-100xP, symbol Switch:SW_MEC_5G
- added J1: USB_A, simpleLED:USB-A-Male, symbol Connector:USB_A
- added SW1: SW_Push, Button_Switch_SMD:SW_SPST_PTS645, symbol Switch:SW_Push
- R1: footprint Resistor_THT:R_Axial_DIN0204_L3.6mm_D1.6mm_P1.90mm_Vertical -> Resistor_THT:R_Axial_DIN0204_L3.6mm_D1.6mm_P5.08mm_Horizontal
Connections:
- net +5V: now also J1.1 (VBUS), SW1.1
- net GND: now also J1.4 (GND)
- net at R1.1: now also SW1.2
- no-connect marks 0 -> 3
Other:
- moved on the sheet: D1, R1

Commit message: updated
Parts:
- D1: footprint Diode_SMD:D_1210_3225Metric_Pad1.42x2.65mm_HandSolder -> LED_THT:LED_D3.0mm
- R1: footprint Resistor_THT:R_Axial_DIN0204_L3.6mm_D1.6mm_P5.08mm_Horizontal -> Resistor_THT:R_Axial_DIN0204_L3.6mm_D1.6mm_P7.62mm_Horizontal
- SW1: footprint Button_Switch_SMD:SW_SPST_PTS645 -> Button_Switch_THT:SW_PUSH_6mm
Other:
- moved on the sheet: D1, J1, R1, SW1
