File: simpleLogicCircuit/simpleLogicCircuit.kicad_pcb (KiCad board)
At the start: 2 copper layers, 100 x 20 mm, 15 parts, among them SW1 SW_Push, SW2 SW_Push

Commit message: updated
Parts:
- removed the REF** at (115.0, 35.0)
- removed the REF** at (20.4, 15.2)
- added REF**: ruler_10cm, simpleLogicCircuit:ruler_10cm, F.Cu at (32.0, 37.0)
- USB-C PWR: renamed from USB C
- moved D1 29.9 mm to (99.8, 51.2)
- moved R2 29.9 mm to (71.1, 53.1)
- moved R3 29.9 mm to (75.1, 53.1)
- moved R4 29.9 mm to (79.1, 53.1)
- moved R5 29.9 mm to (83.1, 53.1)
- moved 74HC00 29.9 mm to (46.4, 60.7)
- moved D2 29.9 mm to (99.8, 59.2)
- moved D3 29.9 mm to (122.8, 55.1)
- moved G*** 29.9 mm to (112.1, 56.4)
- moved R1 29.9 mm to (67.3, 53.1)
- moved SW1 29.9 mm to (88.8, 50.2)
- moved SW2 29.9 mm to (88.8, 58.2)
- moved USB-C PWR 29.9 mm to (32.6, 56.9)
Routing:
- net unconnected-(J1-PadS1): track 0.00 -> 8.60 mm
- net Net-(U1-Pad3): track 15.1 -> 16.3 mm
- net GND: track 45.4 -> 44.7 mm
- net Net-(D2-Pad2): vias 2 -> 1
- removed copper zone on F.Cu, net +5V
- removed copper zone on B.Cu, net GND
Other:
- board size 100 x 20 mm -> 100 x 30 mm
- board text added: "USB-C PWR ONLY"

Commit message: updated
Parts:
- added REF**: keyringhole, simpleLogicCircuit:keyringhole, F.Cu at (128.0, 52.0)
Other:
- outline, holes or cut-outs redrawn
Changed lines of the file:
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@@
     (property "Sheetname" "")
     (attr through_hole)
-    (fp_text reference "D3" (at 1.27 -2.96 90) (layer "F.SilkS")
+    (fp_text reference "D3" (at 1.865 -3.195 90) (layer "F.SilkS")
       (effects (font (size 1 1) (thickness 0.15)))
     )
@@
     )
   )
+  (footprint "simpleLogicCircuit:keyringhole" (layer "F.Cu")
+    (at 128 52)
+    (attr through_hole)
+    (fp_text reference "REF**" (at 0 5 unlocked) (layer "F.SilkS") hide
+      (effects (font (size 1 1) (thickness 0.15)))
+    )
+    (fp_text value "keyringhole" (at 0 6 unlocked) (layer "F.Fab") hide
+      (effects (font (size 1 1) (thickness 0.15)))
+    )
+    (fp_text user "${REFERENCE}" (at 0 9 unlocked) (layer "F.Fab") hide
+      (effects (font (size 1 1) (thickness 0.15)))
+    )
+    (pad "2" thru_hole oval (at 0 0) (size 4 9) (drill oval 3 8) (layers *.Cu *.Mask))
+  )
   (footprint "Button_Switch_THT:SW_PUSH_6mm" (layer "F.Cu")
     (at 88.805 50.16)
@@
     )
   )
-  (gr_rect (start 32 37) (end 132 67) (layer "Edge.Cuts") (width 0.1) (fill none))
+  (gr_arc (start 132 66) (mid 131.707107 66.707107) (end 131 67) (layer "Edge.Cuts") (width 0.1))
+  (gr_line (start 32 66) (end 32 37) (layer "Edge.Cuts") (width 0.1))
+  (gr_line (start 32 37) (end 132 37) (layer "Edge.Cuts") (width 0.1))
+  (gr_arc (start 33 67) (mid 32.292893 66.707107) (end 32 66) (layer "Edge.Cuts") (width 0.1))
+  (gr_line (start 132 37) (end 132 66) (layer "Edge.Cuts") (width 0.1))
+  (gr_line (start 131 67) (end 33 67) (layer "Edge.Cuts") (width 0.1))
   (gr_text "National Institute of Technology, Kagawa College\nDepartment of Electronic Systems Engineering" (at 38 64.5) (layer "F.Cu")
     (effects (font (size 1.2 1.2) (thickness 0.2)) (justify left))
