File: simpleLogicCircuit_v2/simpleLogicCircuit.kicad_pcb (KiCad board)
At the start: 2 copper layers, 100 x 30 mm, 17 parts, among them J1 USB_C_Receptacle_PowerOnly_6P, SW1 SW_Push, SW2 SW_Push, U1 74HC00, X1 LED, X2 LED

Commit message: updated
Parts:
- USB-C PWR: renamed from J1
- renumbered U1 to 74HC00
Routing:
- net /74HC00-4: track 10.9 -> 100.7 mm, vias 0 -> 3
- net /74HC00-13: track 0.00 -> 84.0 mm, vias 0 -> 2
- net /74HC00-2: track 0.00 -> 82.8 mm, vias 0 -> 2
- net /74HC00-5: track 10.7 -> 90.5 mm, vias 0 -> 3
- net /74HC00-11: track 0.00 -> 74.4 mm, vias 0 -> 2
- net /74HC00-3: track 25.1 -> 99.3 mm, vias 0 -> 4
- net /74HC00-6: track 19.0 -> 92.6 mm, vias 0 -> 3
- net /74HC00-12: track 0.00 -> 70.6 mm
- net /74HC00-8: track 9.37 -> 70.3 mm, vias 0 -> 3
- net /74HC00-10: track 20.4 -> 80.4 mm, vias 0 -> 2
- net /74HC00-1: track 13.0 -> 70.8 mm, vias 0 -> 3
- net /74HC00-9: track 9.60 -> 67.2 mm, vias 0 -> 3
- net /X2: track 47.5 -> 72.5 mm, vias 0 -> 4
- net /X1: track 36.2 -> 52.9 mm, vias 0 -> 4
- net /Y: track 47.8 -> 46.3 mm
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- added copper zone on F.Cu, net +5V
- added copper zone on B.Cu, net GND
Other:
- board text added: "+"
- board text added: "1"
- board text added: "10"
- board text added: "11"
- board text added: "12"
- board text added: "13"
- board text added: "14"
- board text added: "2"
- board text added: "3"
- board text added: "4"
- board text added: "5"
- board text added: "6"
- board text added: "7"
- board text added: "8"
- board text added: "9"
- board text added: "USB-C PWR"

Commit message: updated
Parts:
- added 74HC00: 74HC00, Package_DIP:DIP-14_W7.62mm, F.Cu at (45.4, 89.8)
- added 74HC00: 74HC00, Package_DIP:DIP-14_W7.62mm, F.Cu at (45.4, 119.8)
- added AND: Pads_AND, simpleLogicCircuit:pads_of_and, F.Cu at (98.9, 80.5)
- added AND: Pads_AND, simpleLogicCircuit:pads_of_and, F.Cu at (98.9, 110.5)
- added G***: LOGO, simpleLogicCircuit:logo_text_nitkc, B.Cu at (59.1, 43.8)
- added G***: LOGO, simpleLogicCircuit:logo_text_nitkc, B.Cu at (59.1, 103.8)
- added G***: LOGO, simpleLogicCircuit:logo_text_nitkc, B.Cu at (59.1, 73.8)
- added OR: Pads_OR, simpleLogicCircuit:pads_of_or, F.Cu at (98.9, 117.0)
- added OR: Pads_OR, simpleLogicCircuit:pads_of_or, F.Cu at (98.9, 87.0)
- added R1: 10k, Resistor_THT:R_Axial_DIN0204_L3.6mm_D1.6mm_P7.62mm_Horizontal, F.Cu at (73.4, 108.5)
- added R1: 10k, Resistor_THT:R_Axial_DIN0204_L3.6mm_D1.6mm_P7.62mm_Horizontal, F.Cu at (73.4, 78.5)
- added R2: 10k, Resistor_THT:R_Axial_DIN0204_L3.6mm_D1.6mm_P7.62mm_Horizontal, F.Cu at (73.4, 82.4)
- added R2: 10k, Resistor_THT:R_Axial_DIN0204_L3.6mm_D1.6mm_P7.62mm_Horizontal, F.Cu at (73.4, 112.4)
- added R3: R, Resistor_THT:R_Axial_DIN0204_L3.6mm_D1.6mm_P7.62mm_Horizontal, F.Cu at (73.4, 116.0)
- added R3: R, Resistor_THT:R_Axial_DIN0204_L3.6mm_D1.6mm_P7.62mm_Horizontal, F.Cu at (73.4, 86.0)
- added R4: R, Resistor_THT:R_Axial_DIN0204_L3.6mm_D1.6mm_P7.62mm_Horizontal, F.Cu at (73.4, 120.0)
- added R4: R, Resistor_THT:R_Axial_DIN0204_L3.6mm_D1.6mm_P7.62mm_Horizontal, F.Cu at (73.4, 90.0)
- added R5: R, Resistor_THT:R_Axial_DIN0204_L3.6mm_D1.6mm_P7.62mm_Horizontal, F.Cu at (73.4, 123.8)
- added R5: R, Resistor_THT:R_Axial_DIN0204_L3.6mm_D1.6mm_P7.62mm_Horizontal, F.Cu at (73.4, 93.8)
- added REF**: keyringhole, simpleLogicCircuit:keyringhole, F.Cu at (128.0, 112.0)
- added REF**: ruler_10cm, simpleLogicCircuit:ruler_10cm, F.Cu at (32.0, 67.0)
- added REF**: ruler_10cm, simpleLogicCircuit:ruler_10cm, F.Cu at (32.0, 97.0)
- added REF**: keyringhole, simpleLogicCircuit:keyringhole, F.Cu at (128.0, 82.0)
- added SW1: SW_Push, Button_Switch_THT:SW_PUSH_6mm, F.Cu at (77.8, 123.2)
- added SW1: SW_Push, Button_Switch_THT:SW_PUSH_6mm, F.Cu at (77.8, 93.2)
- added SW2: SW_Push, Button_Switch_THT:SW_PUSH_6mm, F.Cu at (87.8, 123.2)
- added SW2: SW_Push, Button_Switch_THT:SW_PUSH_6mm, F.Cu at (87.8, 93.2)
- added USB-C PWR: USB_C_Receptacle_PowerOnly_6P, simpleLogicCircuit:USB-C-A295-CTRPB-1, F.Cu at (31.9, 86.0)
- added USB-C PWR: USB_C_Receptacle_PowerOnly_6P, simpleLogicCircuit:USB-C-A295-CTRPB-1, F.Cu at (31.9, 116.0)
- added X1: LED, LED_THT:LED_D3.0mm, F.Cu at (78.4, 111.3)
- added X1: LED, LED_THT:LED_D3.0mm, F.Cu at (78.4, 81.3)
- added X2: LED, LED_THT:LED_D3.0mm, F.Cu at (84.9, 111.3)
- added X2: LED, LED_THT:LED_D3.0mm, F.Cu at (84.9, 81.3)
- added XOR: Pads_XOR, simpleLogicCircuit:pads_of_xor, F.Cu at (98.9, 123.5)
- added XOR: Pads_XOR, simpleLogicCircuit:pads_of_xor, F.Cu at (98.9, 93.5)
- added Y: LED, LED_THT:LED_D3.0mm, F.Cu at (91.5, 111.3)
- added Y: LED, LED_THT:LED_D3.0mm, F.Cu at (91.5, 81.3)
Routing:
- net /74HC00-4: track 100.7 -> 302.2 mm, vias 3 -> 9
- net /74HC00-3: track 99.3 -> 298.0 mm, vias 4 -> 12
- net /74HC00-6: track 92.6 -> 277.8 mm, vias 3 -> 9
- net /74HC00-5: track 90.5 -> 271.5 mm, vias 3 -> 9
- net /74HC00-13: track 84.0 -> 252.1 mm, vias 2 -> 6
- net +5V: track 83.4 -> 250.1 mm
- net /74HC00-2: track 82.8 -> 248.3 mm, vias 2 -> 6
- net /74HC00-10: track 80.4 -> 241.2 mm, vias 2 -> 6
- net /74HC00-11: track 74.4 -> 223.2 mm, vias 2 -> 6
- net /X2: track 72.5 -> 217.5 mm, vias 4 -> 12
- net /74HC00-1: track 70.8 -> 212.3 mm, vias 3 -> 9
- net /74HC00-12: track 70.6 -> 211.7 mm
- net /74HC00-8: track 70.3 -> 210.9 mm, vias 3 -> 9
- net /74HC00-9: track 67.2 -> 201.5 mm, vias 3 -> 9
- net /X1: track 52.9 -> 158.7 mm, vias 4 -> 12
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Other:
- board size 100 x 30 mm -> 100 x 90 mm
- board text added: "Logic Gate Ruler v1.0 Designed by MILab 2023"
- board text removed: "National Institute of Technology, Kagawa College Department of Electronic Systems Engineering"
