File: simpleLogicCircuit_v1.3/simpleLogicCircuit.kicad_pcb (KiCad board)
At the start: 2 copper layers, 100 x 25 mm, 14 parts, among them J1 USB_C_Receptacle_PowerOnly_6P, SW1 SW_Push, SW2 SW_Push, U1 74HC00

Commit message: Updated
Parts:
- added G***: LOGO, simpleLogicCircuit:logo_text_nitkc, B.Cu at (89.5, 33.8)
- added REF**: keyringhole, simpleLogicCircuit:keyringhole, F.Cu at (135.0, 42.5)
- moved X1 16.0 mm to (86.0, 39.9), turned to 90 degrees
- moved SW1 12.6 mm to (85.2, 50.5), turned to 90 degrees
- moved Y 12.1 mm to (98.0, 39.8), turned to 90 degrees
- moved X2 11.3 mm to (92.0, 39.8), turned to 90 degrees
- moved XOR 8.66 mm to (105.4, 50.6)
- moved OR 8.57 mm to (105.4, 39.4)
- moved AND 8.56 mm to (105.4, 45.0)
- moved R3 7.78 mm to (79.3, 45.4), turned to 180 degrees
- moved R2 6.87 mm to (79.3, 41.5), turned to 180 degrees
- moved R1 6.03 mm to (79.3, 37.6), turned to 180 degrees
- moved 74HC00 5.70 mm to (51.9, 45.3)
- moved SW2 5.33 mm to (94.3, 50.5), turned to 90 degrees
- moved USB-CPWR 1.83 mm to (39.9, 45.0)
- renumbered U1 to 74HC00, J1 to USB-CPWR, D1 to X1, D2 to X2, D3 to Y
Routing:
- net +5V: track 0.00 -> 91.6 mm
- net /74HC00-6: track 0.00 -> 84.8 mm, vias 0 -> 5
- net /74HC00-10: track 0.00 -> 81.7 mm, vias 0 -> 5
- net /74HC00-4: track 0.00 -> 81.5 mm, vias 0 -> 9
- net /74HC00-13: track 0.00 -> 80.1 mm
- net /74HC00-3: track 0.00 -> 78.4 mm, vias 0 -> 6
- net /74HC00-2: track 0.00 -> 77.8 mm, vias 0 -> 4
- net /74HC00-11: track 0.00 -> 76.7 mm
- net /74HC00-8: track 0.00 -> 76.0 mm, vias 0 -> 3
- net /74HC00-9: track 0.00 -> 73.3 mm, vias 0 -> 3
- net /74HC00-12: track 0.00 -> 73.0 mm
- net /74HC00-5: track 0.00 -> 71.5 mm, vias 0 -> 7
- net /74HC00-1: track 0.00 -> 71.2 mm, vias 0 -> 6
- net /Y: track 0.00 -> 44.3 mm, vias 0 -> 5
- net /X1: track 0.00 -> 43.1 mm, vias 0 -> 3
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- added copper zone on F.Cu, net +5V
- added copper zone on B.Cu, net GND
Other:
- board text added: "Logic Gate Ruler v1.3 Designed by MILab 2024"
- board text added: "USB-C POWER"
